File: Regelung_BZSystem/BZ System.sch (EAGLE design)
At the start: 27 parts, among them Q1 Mosfet, U1 ARDUINO-MEGAFULL

Commit message: Neuer Schaltplan
Parts:
- added KOMPRESSOR: 170Ohm, SparkFun-Passives:RESISTORAXIAL-0.3
- added Q2: Mosfet, transistor-fet:BUZ11
- added R6: 1k, SparkFun-Passives:RESISTORAXIAL-0.3
- added R7: 10k, SparkFun-Passives:RESISTORAXIAL-0.3
Connections:
- removed net 3: R4.2
- new net 4: R4.2, U1.4
- new net N$1: Q2.G, R6.1, R7.2
- new net N$4: KOMPRESSOR.2, Q2.D
- new net N$6: R6.2
- new net N$7: KOMPRESSOR.1
- net GND: now also Q2.S, R7.1
Changed lines of the file:
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@@
 <part name="D2" library="diode" deviceset="1N581*" device="" technology="7-B"/>
 <part name="D3" library="diode" deviceset="1N581*" device="" technology="7-B"/>
+<part name="Q2" library="transistor-fet" deviceset="BUZ11" device="" value="Mosfet"/>
+<part name="R6" library="SparkFun-Passives" deviceset="RESISTOR" device="AXIAL-0.3" value="1k"/>
+<part name="GND7" library="SparkFun-Aesthetics" deviceset="GND" device=""/>
+<part name="R7" library="SparkFun-Passives" deviceset="RESISTOR" device="AXIAL-0.3" value="10k"/>
+<part name="KOMPRESSOR" library="SparkFun-Passives" deviceset="RESISTOR" device="AXIAL-0.3" value="170Ohm"/>
+<part name="SUPPLY7" library="SparkFun-Aesthetics" deviceset="12V" device="" value="5V"/>
 </parts>
 <sheets>
@@
 <instance part="D2" gate="G$1" x="17.78" y="40.64" rot="R90"/>
 <instance part="D3" gate="G$1" x="17.78" y="20.32" rot="R90"/>
+<instance part="Q2" gate="G$1" x="256.54" y="76.2"/>
+<instance part="R6" gate="G$1" x="243.84" y="73.66" rot="R180"/>
+<instance part="GND7" gate="1" x="261.62" y="66.04"/>
+<instance part="R7" gate="G$1" x="254" y="71.12" rot="R180"/>
+<instance part="KOMPRESSOR" gate="G$1" x="261.62" y="96.52" rot="R270"/>
+<instance part="SUPPLY7" gate="G$1" x="261.62" y="114.3"/>
 </instances>
 <busses>
@@
 <junction x="60.96" y="35.56"/>
 </segment>
+<segment>
+<pinref part="Q2" gate="G$1" pin="S"/>
+<wire x1="261.62" y1="73.66" x2="261.62" y2="71.12" width="0.1524" layer="91"/>
+<pinref part="GND7" gate="1" pin="GND"/>
+<pinref part="R7" gate="G$1" pin="1"/>
+<wire x1="261.62" y1="71.12" x2="261.62" y2="68.58" width="0.1524" layer="91"/>
+<wire x1="259.08" y1="71.12" x2="261.62" y2="71.12" width="0.1524" layer="91"/>
+<junction x="261.62" y="71.12"/>
+</segment>
 </net>
 <net name="A0" class="0">
@@
 </segment>
 </net>
-<net name="N$1" class="0">
+<net name="KOMPRESSOR" class="0">
 <segment>
 <wire x1="35.56" y1="177.8" x2="35.56" y2="121.92" width="0.1524" layer="91"/>
@@
 <wire x1="223.52" y1="124.46" x2="274.32" y2="124.46" width="0.1524" layer="91"/>
 <wire x1="139.7" y1="76.2" x2="76.2" y2="76.2" width="0.1524" layer="91"/>
-<wire x1="73.66" y1="76.2" x2="0" y2="76.2" width="0.1524" layer="91"/>
-<wire x1="73.66" y1="76.2" x2="76.2" y2="76.2" width="0.1524" layer="91"/>
+<wire x1="76.2" y1="76.2" x2="0" y2="76.2" width="0.1524" layer="91"/>
 <wire x1="76.2" y1="76.2" x2="76.2" y2="0" width="0.1524" layer="91"/>
+<wire x1="223.52" y1="60.96" x2="274.32" y2="60.96" width="0.1524" layer="91"/>
+<label x="259.08" y="60.96" size="1.778" layer="95"/>
 </segment>
 </net>
@@
 <wire x1="162.56" y1="106.68" x2="147.32" y2="106.68" width="0.1524" layer="91"/>
 <label x="147.32" y="106.68" size="1.778" layer="95"/>
-</segment>
-<segment>
-<pinref part="R4" gate="G$1" pin="2"/>
-<wire x1="45.72" y1="66.04" x2="45.72" y2="68.58" width="0.1524" layer="91"/>
-<label x="45.72" y="68.58" size="1.778" layer="95"/>
 </segment>
 </net>
@@
 </segment>
 </net>
+<net name="N$1" class="0">
+<segment>
+<pinref part="R6" gate="G$1" pin="1"/>
+<pinref part="Q2" gate="G$1" pin="G"/>
+<wire x1="248.92" y1="73.66" x2="251.46" y2="73.66" width="0.1524" layer="91"/>
+<pinref part="R7" gate="G$1" pin="2"/>
+<wire x1="248.92" y1="71.12" x2="248.92" y2="73.66" width="0.1524" layer="91"/>
+<junction x="248.92" y="73.66"/>
+</segment>
+</net>
+<net name="N$4" class="0">
+<segment>
+<pinref part="Q2" gate="G$1" pin="D"/>
+<wire x1="261.62" y1="78.74" x2="261.62" y2="91.44" width="0.1524" layer="91"/>
+<pinref part="KOMPRESSOR" gate="G$1" pin="2"/>
+</segment>
+</net>
+<net name="N$6" class="0">
+<segment>
+<pinref part="R6" gate="G$1" pin="2"/>
+<wire x1="238.76" y1="73.66" x2="233.68" y2="73.66" width="0.1524" layer="91"/>
+</segment>
+</net>
+<net name="4" class="0">
+<segment>
+<pinref part="R4" gate="G$1" pin="2"/>
+<wire x1="45.72" y1="66.04" x2="45.72" y2="68.58" width="0.1524" layer="91"/>
+<label x="45.72" y="68.58" size="1.778" layer="95"/>
+<label x="233.68" y="73.66" size="1.778" layer="95"/>
+</segment>
+<segment>
+<pinref part="U1" gate="G$1" pin="4"/>
+<wire x1="162.56" y1="104.14" x2="147.32" y2="104.14" width="0.1524" layer="91"/>
+<label x="147.32" y="104.14" size="1.778" layer="95"/>
+</segment>
+</net>
+<net name="N$7" class="0">
+<segment>
+<pinref part="KOMPRESSOR" gate="G$1" pin="1"/>
+<wire x1="261.62" y1="101.6" x2="261.62" y2="114.3" width="0.1524" layer="91"/>
+<pinref part="SUPPLY7" gate="G$1" pin="12V"/>
+</segment>
+</net>

Commit message: Spannungswandler in Eagle hinzugefügt
Parts:
- added C1, C2: (no value), capacitor-wima:C2,5-3
- added IC1: 7805T, linear:7805T
- KOMPRESSOR: value 170Ohm -> 170
Connections:
- net 12V: now also C2.1, IC1.VI
- net 5V: now also C1.1, IC1.VO
- net GND: now also C1.2, C2.2, IC1.GND
Changed lines of the file:
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@@
 <part name="GND7" library="SparkFun-Aesthetics" deviceset="GND" device=""/>
 <part name="R7" library="SparkFun-Passives" deviceset="RESISTOR" device="AXIAL-0.3" value="10k"/>
-<part name="KOMPRESSOR" library="SparkFun-Passives" deviceset="RESISTOR" device="AXIAL-0.3" value="170Ohm"/>
+<part name="KOMPRESSOR" library="SparkFun-Passives" deviceset="RESISTOR" device="AXIAL-0.3" value="170"/>
 <part name="SUPPLY7" library="SparkFun-Aesthetics" deviceset="12V" device="" value="5V"/>
+<part name="IC1" library="linear" deviceset="78*" device="T" technology="05"/>
+<part name="GND8" library="SparkFun-Aesthetics" deviceset="GND" device=""/>
+<part name="C1" library="capacitor-wima" deviceset="C" device="2,5-3"/>
+<part name="C2" library="capacitor-wima" deviceset="C" device="2,5-3"/>
+<part name="GND9" library="SparkFun-Aesthetics" deviceset="GND" device=""/>
+<part name="GND10" library="SparkFun-Aesthetics" deviceset="GND" device=""/>
+<part name="SUPPLY8" library="SparkFun-Aesthetics" deviceset="12V" device="" value="12V"/>
+<part name="SUPPLY9" library="SparkFun-Aesthetics" deviceset="5V" device="" value="5V (Abgekoppelt von Arduino)"/>
 </parts>
 <sheets>
@@
 <instance part="KOMPRESSOR" gate="G$1" x="261.62" y="96.52" rot="R270"/>
 <instance part="SUPPLY7" gate="G$1" x="261.62" y="114.3"/>
+<instance part="IC1" gate="A1" x="106.68" y="58.42"/>
+<instance part="GND8" gate="1" x="106.68" y="45.72"/>
+<instance part="C1" gate="G$1" x="121.92" y="55.88"/>
+<instance part="C2" gate="G$1" x="88.9" y="55.88"/>
+<instance part="GND9" gate="1" x="88.9" y="45.72"/>
+<instance part="GND10" gate="1" x="121.92" y="45.72"/>
+<instance part="SUPPLY8" gate="G$1" x="83.82" y="63.5"/>
+<instance part="SUPPLY9" gate="G$1" x="132.08" y="63.5"/>
 </instances>
 <busses>
@@
 <junction x="261.62" y="71.12"/>
 </segment>
+<segment>
+<pinref part="IC1" gate="A1" pin="GND"/>
+<pinref part="GND8" gate="1" pin="GND"/>
+<wire x1="106.68" y1="50.8" x2="106.68" y2="48.26" width="0.1524" layer="91"/>
+</segment>
+<segment>
+<pinref part="C2" gate="G$1" pin="2"/>
+<pinref part="GND9" gate="1" pin="GND"/>
+<wire x1="88.9" y1="50.8" x2="88.9" y2="48.26" width="0.1524" layer="91"/>
+</segment>
+<segment>
+<pinref part="C1" gate="G$1" pin="2"/>
+<pinref part="GND10" gate="1" pin="GND"/>
+<wire x1="121.92" y1="50.8" x2="121.92" y2="48.26" width="0.1524" layer="91"/>
+</segment>
 </net>
 <net name="A0" class="0">
@@
 <label x="17.78" y="99.06" size="1.778" layer="95"/>
 </segment>
-</net>
-<net name="KOMPRESSOR" class="0">
+<segment>
+<pinref part="IC1" gate="A1" pin="VO"/>
+<wire x1="116.84" y1="58.42" x2="121.92" y2="58.42" width="0.1524" layer="91"/>
+<pinref part="C1" gate="G$1" pin="1"/>
+<junction x="121.92" y="58.42"/>
+<wire x1="121.92" y1="58.42" x2="132.08" y2="58.42" width="0.1524" layer="91"/>
+<pinref part="SUPPLY9" gate="G$1" pin="5V"/>
+<wire x1="132.08" y1="58.42" x2="132.08" y2="63.5" width="0.1524" layer="91"/>
+</segment>
+</net>
+<net name="SPANNUNGSWANDLER" class="0">
 <segment>
 <wire x1="35.56" y1="177.8" x2="35.56" y2="121.92" width="0.1524" layer="91"/>
@@
 <wire x1="139.7" y1="76.2" x2="76.2" y2="76.2" width="0.1524" layer="91"/>
 <wire x1="76.2" y1="76.2" x2="0" y2="76.2" width="0.1524" layer="91"/>
-<wire x1="76.2" y1="76.2" x2="76.2" y2="0" width="0.1524" layer="91"/>
+<wire x1="76.2" y1="76.2" x2="76.2" y2="40.64" width="0.1524" layer="91"/>
+<wire x1="76.2" y1="40.64" x2="76.2" y2="0" width="0.1524" layer="91"/>
 <wire x1="223.52" y1="60.96" x2="274.32" y2="60.96" width="0.1524" layer="91"/>
 <label x="259.08" y="60.96" size="1.778" layer="95"/>
+<wire x1="76.2" y1="40.64" x2="139.7" y2="40.64" width="0.1524" layer="91"/>
+<wire x1="139.7" y1="40.64" x2="139.7" y2="60.96" width="0.1524" layer="91"/>
+<label x="76.2" y="40.64" size="1.778" layer="95"/>
 </segment>
 </net>
@@
 <wire x1="76.2" y1="109.22" x2="86.36" y2="109.22" width="0.1524" layer="91"/>
 </segment>
-</net>
+<segment>
+<pinref part="IC1" gate="A1" pin="VI"/>
+<wire x1="96.52" y1="58.42" x2="88.9" y2="58.42" width="0.1524" layer="91"/>
+<pinref part="C2" gate="G$1" pin="1"/>
+<wire x1="88.9" y1="58.42" x2="83.82" y2="58.42" width="0.1524" layer="91"/>
+<junction x="88.9" y="58.42"/>
+<pinref part="SUPPLY8" gate="G$1" pin="12V"/>
+<wire x1="83.82" y1="58.42" x2="83.82" y2="63.5" width="0.1524" layer="91"/>
+</segment>
+</net>
